Commit message: successful

File: models/AzureLoong.urdf (robot description, URDF)
Before this commit: robot OpenLoog, 32 links, 31 joints
Joints:
- joint J_ankle_l_pitch: limit lower=-0.43644 upper=0.61087 effort=58.5 velocity=48.8 -> lower=-0.47 upper=0.87 effort=58.5 velocity=48.8
- joint J_ankle_r_pitch: limit lower=-0.43633 upper=0.61087 effort=58.5 velocity=48.8 -> lower=-0.47 upper=0.87 effort=58.5 velocity=48.8
- joint J_arm_l_02: axis -1 0 0 -> 1 0 0
- joint J_hip_l_yaw: origin xyz=0.08225 -0.001 -0.01 rpy=0 0 0 -> xyz=0.08225 0 -0.01 rpy=0 0 0
- joint J_hip_r_yaw: origin xyz=0.08225 -0.001 -0.01 rpy=0 0 0 -> xyz=0.08225 0 -0.01 rpy=0 0 0
- joint J_waist_pitch: origin xyz=0 -0.06525 0 rpy=0 0 0 -> xyz=0 -0.0655 0 rpy=0 0 0
